Commit message: :+1: update laserscan

File: src/hakuroukun_description/urdf/sensors.xacro (robot description, xacro)
@@ -85,9 +85,9 @@
       <parent link="${parent}"/>
       <child link="${lidar_name}"/>
-      <origin xyz="${ox} ${oy} ${oz}"/>
+      <origin xyz="${ox} ${oy} ${oz}" rpy="${roll} ${pitch} ${yaw}"/>
     </joint>
   	<gazebo reference="${lidar_name}">
       <sensor type="ray" name="${lidar_name}">
-        <pose>0 0 0 0 0 0</pose>
+        <pose>0 0 0 0 0 ${yaw}</pose>
         <visualize>false</visualize>
       	<update_rate>${update_rate}</update_rate>

Commit message: :+1: update laserscan

File: src/hakuroukun_description/urdf/sensors.xacro (robot description, xacro)
@@ -74,5 +74,5 @@
           <cylinder length="${length}" radius="${radius}"/>
         </geometry>
-        <origin rpy="${roll} ${pitch} ${yaw}" xyz="0 0 0"/>
+        <origin xyz="0 0 0"/>
         <material name="Black"/>
       </visual>
@@ -89,5 +89,5 @@
   	<gazebo reference="${lidar_name}">
       <sensor type="ray" name="${lidar_name}">
-        <pose>0 0 0 0 0 ${yaw}</pose>
+        <pose>0 0 0 0 0 0</pose>
         <visualize>false</visualize>
       	<update_rate>${update_rate}</update_rate>
