Commit message: :rabbit: change tricycle to ackermann structure

File: src/hakuroukun_description/urdf/actuators_wheels.xacro (robot description, xacro)
@@ -30,8 +30,8 @@
             <actuator name="${name}_motor" >
                 <mechanicalReduction>1.0</mechanicalReduction>
-                <!-- <hardwareInterface>hardware_interface/EffortJointInterface</hardwareInterface> -->
+                <hardwareInterface>hardware_interface/PositionJointInterface</hardwareInterface>
             </actuator>
             <joint name="${parent_link}_to_${name}" type="continuous">
-                <hardwareInterface>hardware_interface/VelocityJointInterface</hardwareInterface>
+                <hardwareInterface>hardware_interface/PositionJointInterface</hardwareInterface>
             </joint>
         </transmission>
@@ -69,8 +69,8 @@
             <actuator name="${name}_motor" >
                 <mechanicalReduction>1.0</mechanicalReduction>
-                <!-- <hardwareInterface>hardware_interface/EffortJointInterface</hardwareInterface> -->
+                <hardwareInterface>hardware_interface/PositionJointInterface</hardwareInterface>
             </actuator>
             <joint name="${parent_link}_to_${name}" type="revolute">
-                <hardwareInterface>hardware_interface/VelocityJointInterface</hardwareInterface>
+                <hardwareInterface>hardware_interface/PositionJointInterface</hardwareInterface>
             </joint>
         </transmission>
@@ -116,5 +116,5 @@
             <actuator name="${name}_motor">
                 <mechanicalReduction>1.0</mechanicalReduction>
-                <!-- <hardwareInterface>hardware_interface/VelocityJointInterface</hardwareInterface> -->
+                <hardwareInterface>hardware_interface/VelocityJointInterface</hardwareInterface>
             </actuator>
         </transmission>
@@ -157,3 +157,46 @@
         </gazebo>
     </xacro:macro>
+    <xacro:macro name="axis_and_wheel" params="name parent_link mass radius thickness x y z mu1 mu2 kp kd file_name">
+        <link name="${name}" >
+            <visual>
+                <geometry>
+                    <mesh filename="${file_name}" scale="0.001 0.001 0.001"/>
+                </geometry>
+                <origin xyz="0.0 0.0 0.0" rpy="0.0 0.0 0.0"/>
+                <material name="White"/>
+            </visual>
+            <collision>
+                <geometry>
+                    <mesh filename="${file_name}" scale="0.001 0.001 0.001"/>
+                </geometry>
+                <origin xyz="0.0 0.0 0.0" rpy="0.0 0.0 0.0"/>
+            </collision>
+            <xacro:inertial_cylinder_y mass="${mass}" radius="${radius}" height="${thickness}" />
+        </link>
+        <gazebo reference="${name}" >
+            <mu1 value="${mu1}"/>
+            <mu2 value="${mu2}"/>
+            <kp value="${kp}" />
+            <kd value="${kd}" />
+        </gazebo>
+        <joint name="${parent_link}_to_${name}" type="continuous">
+            <parent link="${parent_link}"/>
+            <child link="${name}"/>
+            <axis xyz="0 1 0" />
+            <origin xyz="${x} ${y} ${z}" />
+        </joint>
+        <transmission name="${name}_transmission">
+            <type>transmission_interface/SimpleTransmission</type>
+            <joint name="${parent_link}_to_${name}">
+                <hardwareInterface>hardware_interface/VelocityJointInterface</hardwareInterface>
+            </joint>
+            <actuator name="${name}_motor">
+                <mechanicalReduction>1.0</mechanicalReduction>
+                <!-- <hardwareInterface>hardware_interface/VelocityJointInterface</hardwareInterface> -->
+            </actuator>
+        </transmission>
+        <gazebo reference="${name}">
+            <material>Gazebo/Red</material>
+        </gazebo>
+    </xacro:macro>
 </robot>

File: src/hakuroukun_description/urdf/hakuroukun.urdf.xacro (robot description, xacro)
@@ -47,5 +47,5 @@
         <visual>
             <geometry>
-                <mesh filename="package://hakuroukun_description/meshes/base_link.stl" scale="0.001 0.001 0.001"/>
+                <mesh filename="package://hakuroukun_description/meshes/new_base_link.stl" scale="0.001 0.001 0.001"/>
             </geometry>
             <origin rpy="0 0 0" xyz="0 0 0" />
@@ -54,5 +54,5 @@
         <collision>
             <geometry>
-                <mesh filename="package://hakuroukun_description/meshes/base_link.stl" scale="0.001 0.001 0.001"/>
+                <mesh filename="package://hakuroukun_description/meshes/new_base_link.stl" scale="0.001 0.001 0.001"/>
             </geometry>
             <origin rpy="0 0 0" xyz="0 0 0"/>
@@ -82,22 +82,13 @@
         kp="10000000" kd="40"
         file_name="package://hakuroukun_description/meshes/front_wheel.stl" />
-    <xacro:wheel name="rear_left_wheel"
+    <xacro:axis_and_wheel name="rear_wheel"
         parent_link="rear_axis_center"
-        mass="${mass_wheel}"
-        radius="${radius}"
-        thickness="${thickness}"
-        x="0.0" y="0.4" z="0.0"
+        mass="${rear_mass_wheel}"
+        radius="${rear_radius}"
+        thickness="${rear_thickness}"
+        x="0.0" y="0.0" z="0.0"
         mu1="200" mu2="100"
         kp="10000000" kd="40"
-        file_name="package://hakuroukun_description/meshes/rear_left_wheel.stl" />
-    <xacro:wheel name="rear_right_wheel"
-        parent_link="rear_axis_center"
-        mass="${mass_wheel}"
-        radius="${radius}"
-        thickness="${thickness}"
-        x="0.0" y="-0.4" z="0.0"
-        mu1="200" mu2="100"
-        kp="10000000" kd="40"
-        file_name="package://hakuroukun_description/meshes/rear_right_wheel.stl" />
+        file_name="package://hakuroukun_description/meshes/new_rear.stl" />
 <!-- ////////////////////////////// GAZEBO ROS PLUGIN //////////////////////////////////// -->
     <gazebo>

File: src/hakuroukun_description/urdf/properties.xacro (robot description, xacro)
@@ -6,5 +6,5 @@
   <xacro:property name="robot_width" value="0.810" />
   <xacro:property name="robot_height" value="1.070" />
-  <xacro:property name="robot_mass" value="200" />
+  <xacro:property name="robot_mass" value="240" />
   <!-- ///////////////////////////////////////////////////////////// -->
   <!-- /////////////////// Base link to Robot frame /////////////////// -->
@@ -26,3 +26,8 @@
   <xacro:property name="mass_wheel" value="3.803" />
   <!-- ///////////////////////////////////////////////////////////// -->
+    <!-- /////////////////// rear wheels /////////////////// -->
+  <xacro:property name="rear_thickness" value="0.499" />
+  <xacro:property name="rear_radius" value="0.125" />
+  <xacro:property name="rear_mass_wheel" value="17.606" />   <!--3.803+3.803+10-->
+  <!-- ///////////////////////////////////////////////////////////// -->
 </robot>

Commit message: :rabbit: fix robot description

File: src/hakuroukun_description/urdf/actuators_wheels.xacro (robot description, xacro)
@@ -37,5 +37,5 @@
         </transmission>
         <gazebo reference="${name}">
-            <material>Gazebo/Red</material>
+            <material>Gazebo/Grey</material>
         </gazebo>
     </xacro:macro>
@@ -76,5 +76,5 @@
         </transmission>
         <gazebo reference="${name}">
-            <material>Gazebo/Red</material>
+            <material>Gazebo/Grey</material>
         </gazebo>
     </xacro:macro>
@@ -120,5 +120,5 @@
         </transmission>
         <gazebo reference="${name}">
-            <material>Gazebo/Red</material>
+            <material>Gazebo/Grey</material>
         </gazebo>
     </xacro:macro>
@@ -154,5 +154,5 @@
         </joint>
         <gazebo reference="${name}">
-            <material>Gazebo/Red</material>
+            <material>Gazebo/Grey</material>
         </gazebo>
     </xacro:macro>
@@ -193,9 +193,9 @@
             <actuator name="${name}_motor">
                 <mechanicalReduction>1.0</mechanicalReduction>
-                <!-- <hardwareInterface>hardware_interface/VelocityJointInterface</hardwareInterface> -->
-            </actuator>
-        </transmission>
-        <gazebo reference="${name}">
-            <material>Gazebo/Red</material>
+                <hardwareInterface>hardware_interface/VelocityJointInterface</hardwareInterface>
+            </actuator>
+        </transmission>
+        <gazebo reference="${name}">
+            <material>Gazebo/Grey</material>
         </gazebo>
     </xacro:macro>

File: src/hakuroukun_description/urdf/backup/hakuroukun.urdf.xacro (robot description, xacro)
@@ -47,5 +47,5 @@
         <visual>
             <geometry>
-                <mesh filename="package://hakuroukun_description/meshes/new_base_link.stl" scale="0.001 0.001 0.001"/>
+                <mesh filename="package://hakuroukun_description/meshes/base_link.stl" scale="0.001 0.001 0.001"/>
             </geometry>
             <origin rpy="0 0 0" xyz="0 0 0" />
@@ -54,5 +54,5 @@
         <collision>
             <geometry>
-                <mesh filename="package://hakuroukun_description/meshes/new_base_link.stl" scale="0.001 0.001 0.001"/>
+                <mesh filename="package://hakuroukun_description/meshes/base_link.stl" scale="0.001 0.001 0.001"/>
             </geometry>
             <origin rpy="0 0 0" xyz="0 0 0"/>
@@ -60,7 +60,4 @@
         <xacro:inertial_box mass="${robot_mass}" x="${robot_length}" y="${robot_width}" z="${robot_height}" />
     </link>
-    <gazebo reference="robot_frame">
-        <material>Gazebo/Green</material>
-    </gazebo>
     <joint name="base_link_to_robot_frame" type="fixed">
         <parent link="rear_axis_center" />
@@ -85,13 +82,22 @@
         kp="10000000" kd="40"
         file_name="package://hakuroukun_description/meshes/front_wheel.stl" />
-    <xacro:axis_and_wheel name="rear_wheel"
+    <xacro:wheel name="rear_left_wheel"
         parent_link="rear_axis_center"
-        mass="${rear_mass_wheel}"
-        radius="${rear_radius}"
-        thickness="${rear_thickness}"
-        x="0.0" y="0.0" z="0.0"
+        mass="${mass_wheel}"
+        radius="${radius}"
+        thickness="${thickness}"
+        x="0.0" y="0.4" z="0.0"
         mu1="200" mu2="100"
         kp="10000000" kd="40"
-        file_name="package://hakuroukun_description/meshes/new_rear.stl" />
+        file_name="package://hakuroukun_description/meshes/rear_left_wheel.stl" />
+    <xacro:wheel name="rear_right_wheel"
+        parent_link="rear_axis_center"
+        mass="${mass_wheel}"
+        radius="${radius}"
+        thickness="${thickness}"
+        x="0.0" y="-0.4" z="0.0"
+        mu1="200" mu2="100"
+        kp="10000000" kd="40"
+        file_name="package://hakuroukun_description/meshes/rear_right_wheel.stl" />
 <!-- ////////////////////////////// GAZEBO ROS PLUGIN //////////////////////////////////// -->
     <gazebo>

Commit message: :+1: implement hakuroukun steering controllers

File: src/hakuroukun_description/urdf/actuators_wheels.xacro (robot description, xacro)
@@ -146,5 +146,5 @@
             <kd value="${kd}" />
         </gazebo>
-        <joint name="${parent_link}_to_${name}" type="continuous">
+        <joint name="${parent_link}_to_${name}" type="fixed">
             <parent link="${parent_link}"/>
             <child link="${name}"/>

File: src/hakuroukun_description/urdf/hakuroukun.urdf.xacro (robot description, xacro)
@@ -97,5 +97,4 @@
     <gazebo>
         <plugin name="gazebo_ros_control" filename="libgazebo_ros_control.so">
-            <robotNamespace>hakuroukun</robotNamespace>
             <robotSimType>gazebo_ros_control/DefaultRobotHWSim</robotSimType>
             <legacyModeNS>false</legacyModeNS>

Commit message: :+1: implement hakuroukun steering controllers

File: src/hakuroukun_description/urdf/actuators_wheels.xacro (robot description, xacro)
@@ -146,5 +146,5 @@
             <kd value="${kd}" />
         </gazebo>
-        <joint name="${parent_link}_to_${name}" type="fixed">
+        <joint name="${parent_link}_to_${name}" type="continuous">
             <parent link="${parent_link}"/>
             <child link="${name}"/>
@@ -153,4 +153,14 @@
             <!-- <dynamics damping="0.0" friction="0.0"/> -->
         </joint>
+        <transmission name="${name}_transmission">
+            <type>transmission_interface/SimpleTransmission</type>
+            <joint name="${parent_link}_to_${name}">
+                <hardwareInterface>hardware_interface/VelocityJointInterface</hardwareInterface>
+            </joint>
+            <actuator name="${name}_motor">
+                <mechanicalReduction>1.0</mechanicalReduction>
+                <hardwareInterface>hardware_interface/VelocityJointInterface</hardwareInterface>
+            </actuator>
+        </transmission>
         <gazebo reference="${name}">
             <material>Gazebo/Grey</material>

Commit message: :+1: update sensors gps

File: src/hakuroukun_description/urdf/actuators_wheels.xacro (robot description, xacro)
@@ -196,5 +196,5 @@
             <origin xyz="${x} ${y} ${z}" />
         </joint>
-        <transmission name="${name}_transmission">
+        <!-- <transmission name="${name}_transmission">
             <type>transmission_interface/SimpleTransmission</type>
             <joint name="${parent_link}_to_${name}">
@@ -205,5 +205,5 @@
                 <hardwareInterface>hardware_interface/VelocityJointInterface</hardwareInterface>
             </actuator>
-        </transmission>
+        </transmission>  -->
         <gazebo reference="${name}">
             <material>Gazebo/Grey</material>

File: src/hakuroukun_description/urdf/hakuroukun.urdf.xacro (robot description, xacro)
@@ -9,4 +9,6 @@
     <!-- Import wheels and actuator properties -->
     <xacro:include filename="$(find hakuroukun_description)/urdf/actuators_wheels.xacro" />
+    <!-- Import sensors -->
+    <xacro:include filename="$(find hakuroukun_description)/urdf/sensors.xacro" />
     <xacro:property name="robot_namespace" value="hakuroukun"/>
     <!-- Base link-->
@@ -73,5 +75,5 @@
         mass="${mass_steering_unit}"
         size_x="${steering_X}"  size_y="${steering_Y}" size_z="${steering_Z}"
-        x="${rear_axis_center_to_steering_center}" y="-0.01" z="0.0"
+        x="${rear_axis_center_to_steering_center}" y="-0.01" z="-0.02"
         file_name="package://hakuroukun_description/meshes/steering.stl" />
 <!-- ///////////////////////////////////////// WHEELS //////////////////////////////////// -->
@@ -82,6 +84,6 @@
         thickness="${thickness}"
         x="0.0" y="0.0" z="0.0"
-        mu1="200" mu2="100"
-        kp="50000" kd="40"
+        mu1="0.6" mu2="0.6"
+        kp="10000000" kd="40"
         file_name="package://hakuroukun_description/meshes/front_wheel.stl" />
     <xacro:axis_and_wheel name="rear_wheel"
@@ -90,8 +92,10 @@
         radius="${rear_radius}"
         thickness="${rear_thickness}"
-        x="0.0" y="0.0" z="0.0"
-        mu1="200" mu2="100"
-        kp="50000" kd="40"
+        x="0.0" y="0.0" z="-0.02"
+        mu1="0.6" mu2="0.6"
+        kp="10000000" kd="40"
         file_name="package://hakuroukun_description/meshes/new_rear.stl" />
+    <xacro:imu_sensor parent="base_link" imu_name="imu" imu_topic="imu/data_raw" mass="${imu_mass}" sizex="0.03" sizey="0.03" sizez="0.005" ox="0.0" oy="0.0" oz="0.01" update_rate="${imu_update_rate}" noise="${imu_noise}" />
+    <xacro:gps_sensor parent="base_link" gps_name="gps" gps_topic="gps/fix" mass="${gps_mass}" sizex="0.03" sizey="0.03" sizez="0.005" ox="0.0" oy="0.0" oz="0.0015" update_rate="${gps_update_rate}" initial_latitude="${gps_latitude}" initial_longitude="${gps_longitude}" noise="${gps_noise}" />
 <!-- ////////////////////////////// GAZEBO ROS PLUGIN //////////////////////////////////// -->
     <gazebo>

File: src/hakuroukun_description/urdf/properties.xacro (robot description, xacro)
@@ -6,5 +6,5 @@
   <xacro:property name="robot_width" value="0.810" />
   <xacro:property name="robot_height" value="1.070" />
-  <xacro:property name="robot_mass" value="140" />
+  <xacro:property name="robot_mass" value="50" />
   <!-- ///////////////////////////////////////////////////////////// -->
   <!-- /////////////////// Base link to Robot frame /////////////////// -->
@@ -31,3 +31,11 @@
   <xacro:property name="rear_mass_wheel" value="17.606" />   <!--3.803+3.803+10-->
   <!-- ///////////////////////////////////////////////////////////// -->
+  <xacro:property name="imu_update_rate" value="40.0" />
+  <xacro:property name="imu_mass" value="0.05" />
+  <xacro:property name="imu_noise" value="0.001" />
+  <xacro:property name="gps_update_rate" value="10.0" />
+  <xacro:property name="gps_mass" value="0.05" />
+  <xacro:property name="gps_noise" value="0.001" />
+  <xacro:property name="gps_latitude" value="34.835190564394" />
+  <xacro:property name="gps_longitude" value="137.45711512765206" />
 </robot>
