Commit message: modify to adapt with tasp with cones

File: src/hakuroukun_description/urdf/actuators_wheels.xacro (robot description, xacro)
@@ -87,5 +87,5 @@
                 </geometry>
                 <origin xyz="0.0 0.0 0.0" rpy="0.0 0.0 0.0"/>
-                <material name="White"/>
+                <material name="DarkGrey"/>
             </visual>
             <collision>
@@ -120,5 +120,5 @@
         </transmission>
         <gazebo reference="${name}">
-            <material>Gazebo/Grey</material>
+            <material>Gazebo/DarkGrey</material>
         </gazebo>
     </xacro:macro>
@@ -130,5 +130,5 @@
                 </geometry>
                 <origin xyz="0.0 0.0 0.0" rpy="0.0 0.0 0.0"/>
-                <material name="White"/>
+                <material name="DarkGrey"/>
             </visual>
             <collision>
@@ -164,5 +164,5 @@
         </transmission>
         <gazebo reference="${name}">
-            <material>Gazebo/Grey</material>
+            <material>Gazebo/DarkGrey</material>
         </gazebo>
     </xacro:macro>
@@ -174,5 +174,5 @@
                 </geometry>
                 <origin xyz="0.0 0.0 0.0" rpy="0.0 0.0 0.0"/>
-                <material name="White"/>
+                <material name="DarkGrey"/>
             </visual>
             <collision>
@@ -207,5 +207,5 @@
         </transmission>  -->
         <gazebo reference="${name}">
-            <material>Gazebo/Grey</material>
+            <material>Gazebo/DarkGrey</material>
         </gazebo>
     </xacro:macro>

File: src/hakuroukun_description/urdf/colors.xacro (robot description, xacro)
@@ -19,5 +19,5 @@
         <color rgba="0.75 0.75 0.75 1"/>
     </material>
-    <material name="Darkgrey">
+    <material name="DarkGrey">
         <color rgba="0.41 0.41 0.41 1"/>
     </material>

File: src/hakuroukun_description/urdf/hakuroukun.urdf.xacro (robot description, xacro)
@@ -70,4 +70,21 @@
         <origin xyz="${base_link_to_robot_frame_X} ${base_link_to_robot_frame_Y} ${base_link_to_robot_frame_Z}" />
     </joint>
+    <!-- lidar center-->
+    <link name="lidar_center">
+        <visual>
+        <geometry>
+            <box size="0.01 0.01 0.01"/>
+        </geometry>
+        <material name="Red"/>
+        </visual>
+    </link>
+    <gazebo reference="lidar_center">
+        <material>Gazebo/Red</material>
+    </gazebo>
+    <joint name="rear_axis_center_to_lidar_center" type="fixed">
+        <parent link="rear_axis_center" />
+        <child link="lidar_center" />
+        <origin xyz="1.03 0.0 ${0.365-rear_radius}" />
+    </joint>
 <!-- ///////////////////////////////////////// STEERING //////////////////////////////////// -->
     <xacro:steering_continuous name="front_wheel_shaft"
@@ -84,5 +101,5 @@
         thickness="${thickness}"
         x="0.0" y="0.0" z="0.0"
-        mu1="0.6" mu2="0.6"
+        mu1="0.7" mu2="0.7"
         kp="10000000" kd="40"
         file_name="package://hakuroukun_description/meshes/front_wheel.stl" />
@@ -93,18 +110,17 @@
         thickness="${rear_thickness}"
         x="0.0" y="0.0" z="-0.02"
-        mu1="0.6" mu2="0.6"
+        mu1="0.7" mu2="0.7"
         kp="10000000" kd="40"
         file_name="package://hakuroukun_description/meshes/new_rear.stl" />
-    <xacro:imu_sensor parent="rear_axis_center" imu_name="imu" imu_topic="imu/data_raw" mass="${imu_mass}" sizex="0.03" sizey="0.03" sizez="0.005" ox="0.62" oy="-0.25" oz="1.00" update_rate="${imu_update_rate}" noise="${imu_noise}" />
-    <xacro:gps_sensor parent="rear_axis_center" gps_name="gps" gps_topic="fix" mass="${gps_mass}" sizex="0.03" sizey="0.03" sizez="0.005" ox="0.6" oy="0.0" oz="1.365" update_rate="${gps_update_rate}" initial_latitude="${gps_latitude}" initial_longitude="${gps_longitude}" noise="${gps_noise}" />
-    <xacro:lidar_sensor parent="rear_axis_center" lidar_name="right_lidar" length="${lidar_length}" radius="${lidar_radius}" mass="${lidar_mass}" ox="1.05" oy="-0.33" oz="0.3" roll="0" pitch="0" yaw="${pi}" update_rate="${lidar_update_rate}" min_angle="${lidar_min_angle}" max_angle="${lidar_max_angle}" min_range="${lidar_min_range}" max_range="${lidar_max_range}" range_resolution="${lidar_range_resolution}" stdv="${lidar_stdv}" />
-    <xacro:lidar_sensor parent="rear_axis_center" lidar_name="left_lidar" length="${lidar_length}" radius="${lidar_radius}" mass="${lidar_mass}" ox="1.05" oy="0.33" oz="0.3" roll="0" pitch="0" yaw="${pi}" update_rate="${lidar_update_rate}" min_angle="${lidar_min_angle}" max_angle="${lidar_max_angle}" min_range="${lidar_min_range}" max_range="${lidar_max_range}" range_resolution="${lidar_range_resolution}" stdv="${lidar_stdv}" />
+    <xacro:imu_sensor parent="rear_axis_center" imu_name="imu" imu_topic="imu/data_raw" mass="${imu_mass}" sizex="0.03" sizey="0.03" sizez="0.005" ox="0.62" oy="-0.25" oz="${1.00-rear_radius}" update_rate="${imu_update_rate}" noise="${imu_noise}" />
+    <xacro:gps_sensor parent="rear_axis_center" gps_name="gps" gps_topic="fix" mass="${gps_mass}" sizex="0.03" sizey="0.03" sizez="0.005" ox="0.6" oy="0.0" oz="${1.365-rear_radius}" update_rate="${gps_update_rate}" initial_latitude="${gps_latitude}" initial_longitude="${gps_longitude}" noise="${gps_noise}" />
+    <xacro:lidar_sensor parent="rear_axis_center" lidar_name="right_lidar" length="${lidar_length}" radius="${lidar_radius}" mass="${lidar_mass}" ox="1.03" oy="-0.31" oz="${0.365-rear_radius}" roll="0" pitch="0" yaw="${pi}" update_rate="${lidar_update_rate}" min_angle="${lidar_min_angle}" max_angle="${lidar_max_angle}" min_range="${lidar_min_range}" max_range="${lidar_max_range}" range_resolution="${lidar_range_resolution}" stdv="${lidar_stdv}" />
+    <xacro:lidar_sensor parent="rear_axis_center" lidar_name="left_lidar" length="${lidar_length}" radius="${lidar_radius}" mass="${lidar_mass}" ox="1.03" oy="0.31" oz="${0.365-rear_radius}" roll="0" pitch="0" yaw="${pi}" update_rate="${lidar_update_rate}" min_angle="${lidar_min_angle}" max_angle="${lidar_max_angle}" min_range="${lidar_min_range}" max_range="${lidar_max_range}" range_resolution="${lidar_range_resolution}" stdv="${lidar_stdv}" />
     <xacro:ground_truth parent="base_link" sizex="0.01" sizey="0.01" sizez="0.01" ox="0.0" oy="0.0" oz="0.01" mass="1"/>
-    <xacro:camera_sensor parent="rear_axis_center" camera_name="camera" mass="0.1" sizex="0.03" sizey="0.1" sizez="0.03" ox="1.2" oy="0.0" oz="0.8"/>
-<!-- ////////////////////////////// GAZEBO ROS PLUGIN //////////////////////////////////// -->
+    <xacro:zed2_camera camera_name="camera_link" parent="rear_axis_center" mass="0.06" ox="1.01" oy="0.0" oz="${1.195-rear_radius}" roll="0" pitch="0" yaw="0" />
+    <!-- ////////////////////////////// GAZEBO ROS PLUGIN //////////////////////////////////// -->
     <gazebo>
         <plugin name="gazebo_ros_control" filename="libgazebo_ros_control.so">
-            <robotSimType>gazebo_ros_control/DefaultRobotHWSim</robotSimType>
-            <legacyModeNS>false</legacyModeNS>
+            <robotNamespace>/</robotNamespace>
         </plugin>
     </gazebo>

File: src/hakuroukun_description/urdf/properties.xacro (robot description, xacro)
@@ -1,10 +1,10 @@
 <?xml version="1.0"?>
 <robot name="musashi_robot" xmlns:xacro="http://ros.org/wiki/xacro">
-  <xacro:property name="pi" value="3.14159" />
+  <!-- <xacro:property name="pi" value="3.14159" /> -->
   <!-- /////////////////// Robot Main /////////////////// -->
   <xacro:property name="robot_length" value="1.430" />
   <xacro:property name="robot_width" value="0.810" />
   <xacro:property name="robot_height" value="1.070" />
-  <xacro:property name="robot_mass" value="50" />
+  <xacro:property name="robot_mass" value="270" />
   <!-- ///////////////////////////////////////////////////////////// -->
   <!-- /////////////////// Base link to Robot frame /////////////////// -->
@@ -17,5 +17,5 @@
   <xacro:property name="steering_Y" value="0.2" />
   <xacro:property name="steering_Z" value="0.2" />
-  <xacro:property name="mass_steering_unit" value="2" />
+  <xacro:property name="mass_steering_unit" value="4" />
   <xacro:property name="upper_limit" value="1.5708" />
   <xacro:property name="lower_limit" value="-1.5708" />
@@ -33,19 +33,19 @@
   <xacro:property name="imu_update_rate" value="40.0" />
   <xacro:property name="imu_mass" value="0.05" />
-  <xacro:property name="imu_noise" value="0.01" />
-  <xacro:property name="gps_update_rate" value="10.0" />
+  <xacro:property name="imu_noise" value="0.0" />
+  <xacro:property name="gps_update_rate" value="40.0" />
   <xacro:property name="gps_mass" value="0.05" />
-  <xacro:property name="gps_noise" value="0.01" />
+  <xacro:property name="gps_noise" value="0.0" />
   <xacro:property name="gps_latitude" value="34.70242845166667" />
   <xacro:property name="gps_longitude" value="137.408935105" />
-  <xacro:property name="lidar_update_rate" value="10.0" />			<!-- update rate in ms or in Hz??? -->
-  <xacro:property name="lidar_mass" value="0.3" />
-  <xacro:property name="lidar_length" value="0.04" />
-  <xacro:property name="lidar_radius" value="0.0325" />
-  <xacro:property name="lidar_min_range" value="0.15" />
+  <xacro:property name="lidar_update_rate" value="15" />			<!-- Hz -->
+  <xacro:property name="lidar_mass" value="0.19" />
+  <xacro:property name="lidar_length" value="0.041" />
+  <xacro:property name="lidar_radius" value="0.038" />
+  <xacro:property name="lidar_min_range" value="0.2" />
   <xacro:property name="lidar_max_range" value="8.0" />
   <xacro:property name="lidar_stdv" value="0.01" />
   <xacro:property name="lidar_range_resolution" value="0.01" />
-  <xacro:property name="lidar_min_angle" value="0.0" />
-  <xacro:property name="lidar_max_angle" value="6.283185" />
+  <xacro:property name="lidar_min_angle" value="${-2*pi}" />
+  <xacro:property name="lidar_max_angle" value="${2*pi}" />
 </robot>

File: src/hakuroukun_description/urdf/sensors.xacro (robot description, xacro)
@@ -7,5 +7,5 @@
           <box size="${sizex} ${sizey} ${sizez}"/>
         </geometry>
-        <material name="White"/>
+        <material name="Grey"/>
       </visual>
       <xacro:inertial_box mass="${mass}" x="${sizex}" y="${sizey}" z="${sizez}" />
@@ -17,5 +17,5 @@
     </joint>
     <gazebo reference="${imu_name}">
-      <material>Gazebo/White</material>
+      <material>Gazebo/Grey</material>
       <gravity>true</gravity>
       <sensor name="${imu_name}_sensor" type="imu">
@@ -44,8 +44,11 @@
 	      <box size="${sizex} ${sizey} ${sizez}"/>
 		</geometry>
-		<material name="White"/>
+		<material name="Grey"/>
 	  </visual>
 	  <xacro:inertial_box mass="${mass}" x="${sizex}" y="${sizey}" z="${sizez}" />
 	</link>
+  <gazebo reference="${gps_name}">
+    <material>Gazebo/Grey</material>
+  </gazebo>
 	<joint name="${parent}_to_${gps_name}" type="fixed">
 	  <parent link="${parent}"/>
@@ -74,11 +77,11 @@
           <cylinder length="${length}" radius="${radius}"/>
         </geometry>
-        <origin xyz="0 0 0"/>
-        <material name="Black"/>
+        <origin xyz="0 0 0.05"/>
+        <material name="DarkGrey"/>
       </visual>
       <xacro:inertial_cylinder_z mass="${mass}" radius="${radius}" height="${length}" />
     </link>
     <gazebo reference="${lidar_name}">
-      <material>Gazebo/Black</material>
+      <material>Gazebo/DarkGrey</material>
   	</gazebo>
     <joint name="$[parent}_to_${lidar_name}" type="fixed">
@@ -95,5 +98,5 @@
           <scan>
             <horizontal>
-              <samples>400</samples>
+              <samples>360</samples>
               <resolution>1</resolution>
               <min_angle>${min_angle}</min_angle>
@@ -147,44 +150,37 @@
     </gazebo>
   </xacro:macro>
-  <xacro:macro name="camera_sensor" params="parent camera_name mass ox oy oz sizex sizey sizez">
+  <xacro:macro name="zed2_camera" params="camera_name parent mass ox oy oz roll pitch yaw">
+    <!-- Define the camera link -->
     <link name="${camera_name}">
-      <visual>
-        <geometry>
-          <box size="${sizex} ${sizey} ${sizez}"/>
-        </geometry>
-        <material name="White"/>
-      </visual>
-      <xacro:inertial_box mass="${mass}" x="${sizex}" y="${sizey}" z="${sizez}" />
+        <!-- Visual representation -->
+        <visual>
+            <geometry>
+                <mesh filename="package://hakuroukun_description/meshes/ZED2.stl" scale="0.001 0.001 0.001"/>
+            </geometry>
+            <origin xyz="0 0 0" rpy="0 0 ${-pi/2}"/>
+            <material name="DarkGrey"/>
+        </visual>
+        <!-- Collision representation -->
+        <collision>
+            <geometry>
+                <mesh filename="package://hakuroukun_description/meshes/ZED2.stl" scale="0.001 0.001 0.001"/>
+            </geometry>
+            <origin xyz="0 0 0" rpy="0 0 ${-pi/2}"/>
+        </collision>
+        <!-- Inertial properties -->
+        <inertial>
+            <origin xyz="0 0 0" rpy="0 0 0"/>
+            <mass value="${mass}"/>
+            <inertia ixx="0.001" ixy="0.0" ixz="0.0" iyy="0.001" iyz="0.0" izz="0.001"/>
+        </inertial>
     </link>
+    <!-- Joint connecting the camera to the parent link -->
     <joint name="${parent}_to_${camera_name}" type="fixed">
-      <parent link="${parent}"/>
-      <child link="${camera_name}"/>
-      <origin xyz="${ox} ${oy} ${oz}"/>
+        <parent link="${parent}"/>
+        <child link="${camera_name}"/>
+        <origin xyz="${ox} ${oy} ${oz}" rpy="${roll} ${pitch} ${yaw}"/>
     </joint>
     <gazebo reference="${camera_name}">
-       <sensor type="camera" name="${camera_name}_camera">
-        <always_on>true</always_on>
-        <update_rate>30.0</update_rate>
-        <visualize>true</visualize>
-        <camera name="${camera_name}_camera">
-          <horizontal_fov>1.3962634</horizontal_fov>
-          <image>
-            <width>640</width>
-            <height>480</height>
-            <format>R8G8B8</format>
-          </image>
-          <clip>
-            <near>0.1</near>
-            <far>100</far>
-          </clip>
-        </camera>
-        <plugin name="camera_controller" filename="libgazebo_ros_camera.so">
-          <updateRate>30.0</updateRate>
-          <cameraName>${camera_name}_camera</cameraName>
-          <imageTopicName>${camera_name}/image_raw</imageTopicName>
-          <cameraInfoTopicName>${camera_name}/camera_info</cameraInfoTopicName>
-          <frameName>${camera_name}</frameName>
-        </plugin>
-      </sensor>
+        <material>Gazebo/DarkGrey</material>
     </gazebo>
   </xacro:macro>
