Commit message: :+1: integrate hakuroukun control with gazebo

File: src/hakuroukun_description/urdf/hakuroukun.urdf.xacro (robot description, xacro)
@@ -83,5 +83,5 @@
         x="0.0" y="0.0" z="0.0"
         mu1="200" mu2="100"
-        kp="10000000" kd="40"
+        kp="50000" kd="40"
         file_name="package://hakuroukun_description/meshes/front_wheel.stl" />
     <xacro:axis_and_wheel name="rear_wheel"
@@ -92,5 +92,5 @@
         x="0.0" y="0.0" z="0.0"
         mu1="200" mu2="100"
-        kp="10000000" kd="40"
+        kp="50000" kd="40"
         file_name="package://hakuroukun_description/meshes/new_rear.stl" />
 <!-- ////////////////////////////// GAZEBO ROS PLUGIN //////////////////////////////////// -->

File: src/hakuroukun_description/urdf/properties.xacro (robot description, xacro)
@@ -6,5 +6,5 @@
   <xacro:property name="robot_width" value="0.810" />
   <xacro:property name="robot_height" value="1.070" />
-  <xacro:property name="robot_mass" value="240" />
+  <xacro:property name="robot_mass" value="140" />
   <!-- ///////////////////////////////////////////////////////////// -->
   <!-- /////////////////// Base link to Robot frame /////////////////// -->

Commit message: :+1: update lidar

File: src/hakuroukun_description/urdf/hakuroukun.urdf.xacro (robot description, xacro)
@@ -14,5 +14,5 @@
     <!-- Base link-->
     <link name="base_link">
-        <!-- <visual>
+        <visual>
             <geometry>
                 <box size="0.01 0.01 0.01"/>
@@ -23,5 +23,5 @@
                 <box size="0.01 0.01 0.01"/>
             </geometry>
-        </collision> -->
+        </collision>
     </link>
     <gazebo reference="base_link">
@@ -96,6 +96,8 @@
         kp="10000000" kd="40"
         file_name="package://hakuroukun_description/meshes/new_rear.stl" />
-    <xacro:imu_sensor parent="base_link" imu_name="imu" imu_topic="imu/data_raw" mass="${imu_mass}" sizex="0.03" sizey="0.03" sizez="0.005" ox="0.0" oy="0.0" oz="0.01" update_rate="${imu_update_rate}" noise="${imu_noise}" />
-    <xacro:gps_sensor parent="base_link" gps_name="gps" gps_topic="gps/fix" mass="${gps_mass}" sizex="0.03" sizey="0.03" sizez="0.005" ox="0.0" oy="0.0" oz="0.0015" update_rate="${gps_update_rate}" initial_latitude="${gps_latitude}" initial_longitude="${gps_longitude}" noise="${gps_noise}" />
+    <xacro:imu_sensor parent="rear_axis_center" imu_name="imu" imu_topic="imu/data_raw" mass="${imu_mass}" sizex="0.03" sizey="0.03" sizez="0.005" ox="0.6" oy="0.0" oz="1.365" update_rate="${imu_update_rate}" noise="${imu_noise}" />
+    <xacro:gps_sensor parent="rear_axis_center" gps_name="gps" gps_topic="gps/fix" mass="${gps_mass}" sizex="0.03" sizey="0.03" sizez="0.005" ox="0.62" oy="0.25" oz="1.00" update_rate="${gps_update_rate}" initial_latitude="${gps_latitude}" initial_longitude="${gps_longitude}" noise="${gps_noise}" />
+    <xacro:lidar_sensor parent="rear_axis_center" lidar_name="right_lidar" length="${lidar_length}" radius="${lidar_radius}" mass="${lidar_mass}" ox="1.05" oy="-0.33" oz="0.3" update_rate="${lidar_update_rate}" min_angle="${lidar_min_angle}" max_angle="${lidar_max_angle}" min_range="${lidar_min_range}" max_range="${lidar_max_range}" range_resolution="${lidar_range_resolution}" stdv="${lidar_stdv}" />
+    <xacro:lidar_sensor parent="rear_axis_center" lidar_name="left_lidar" length="${lidar_length}" radius="${lidar_radius}" mass="${lidar_mass}" ox="1.05" oy="0.33" oz="0.3" update_rate="${lidar_update_rate}" min_angle="${lidar_min_angle}" max_angle="${lidar_max_angle}" min_range="${lidar_min_range}" max_range="${lidar_max_range}" range_resolution="${lidar_range_resolution}" stdv="${lidar_stdv}" />
 <!-- ////////////////////////////// GAZEBO ROS PLUGIN //////////////////////////////////// -->
     <gazebo>

File: src/hakuroukun_description/urdf/properties.xacro (robot description, xacro)
@@ -39,3 +39,13 @@
   <xacro:property name="gps_latitude" value="34.835190564394" />
   <xacro:property name="gps_longitude" value="137.45711512765206" />
+  <xacro:property name="lidar_update_rate" value="10.0" />			<!-- update rate in ms or in Hz??? -->
+  <xacro:property name="lidar_mass" value="0.3" />
+  <xacro:property name="lidar_length" value="0.04" />
+  <xacro:property name="lidar_radius" value="0.0325" />
+  <xacro:property name="lidar_min_range" value="0.15" />
+  <xacro:property name="lidar_max_range" value="8.0" />
+  <xacro:property name="lidar_stdv" value="0.01" />
+  <xacro:property name="lidar_range_resolution" value="0.01" />
+  <xacro:property name="lidar_min_angle" value="0.0" />
+  <xacro:property name="lidar_max_angle" value="6.283185" />
 </robot>

File: src/hakuroukun_description/urdf/sensors.xacro (robot description, xacro)
@@ -67,3 +67,58 @@
 	</gazebo>
 	</xacro:macro>
+  <xacro:macro name="lidar_sensor" params="parent lidar_name length radius mass ox oy oz update_rate min_angle max_angle min_range max_range range_resolution stdv" >
+    <link name="${lidar_name}">
+      <visual>
+        <geometry>
+          <cylinder length="${length}" radius="${radius}"/>
+        </geometry>
+        <origin rpy="0 0 0" xyz="0 0 0"/>
+        <material name="Black"/>
+      </visual>
+      <xacro:inertial_cylinder_z mass="${mass}" radius="${radius}" height="${length}" />
+    </link>
+    <gazebo reference="${lidar_name}">
+      <material>Gazebo/Black</material>
+  	</gazebo>
+    <joint name="$[parent}_to_${lidar_name}" type="fixed">
+      <parent link="${parent}"/>
+        <child link="${lidar_name}"/>
+      <origin xyz="${ox} ${oy} ${oz}"/>
+    </joint>
+  	<gazebo reference="${lidar_name}">
+      <sensor type="ray" name="rplidar_sensor">
+        <pose>0 0 0 0 0 0</pose>
+        <visualize>false</visualize>
+      	<update_rate>${update_rate}</update_rate>
+      	<ray>
+          <scan>
+            <horizontal>
+              <samples>400</samples>
+              <resolution>1</resolution>
+              <min_angle>${min_angle}</min_angle>
+              <max_angle>${max_angle}</max_angle>
+          	</horizontal>
+          </scan>
+          <range>
+            <min>${min_range}</min>
+            <max>${max_range}</max>
+          	<resolution>${range_resolution}</resolution>
+          </range>
+          <noise>
+            <type>gaussian</type>
+          	<!-- Noise parameters based on published spec for Hokuyo laser
+               	achieving "+-30mm" accuracy at range < 10m.  A mean of 0.0m and
+               	stddev of 0.01m will put 99.7% of samples within 0.03m of the true
+               	reading. -->
+          	<mean>0.0</mean>
+          	<stddev>${stdv}</stddev>
+          </noise>
+      	</ray>
+      	<plugin name="lidar_controller" filename="libgazebo_ros_laser.so">
+          <topicName>${lidar_name}/scan</topicName>
+          <frameName>${lidar_name}</frameName>
+      	</plugin>
+      </sensor>
+    </gazebo>
+  </xacro:macro>
 </robot>

Commit message: :+1: update localization method

File: src/hakuroukun_description/urdf/hakuroukun.urdf.xacro (robot description, xacro)
@@ -96,6 +96,6 @@
         kp="10000000" kd="40"
         file_name="package://hakuroukun_description/meshes/new_rear.stl" />
-    <xacro:imu_sensor parent="rear_axis_center" imu_name="imu" imu_topic="imu/data_raw" mass="${imu_mass}" sizex="0.03" sizey="0.03" sizez="0.005" ox="0.6" oy="0.0" oz="1.365" update_rate="${imu_update_rate}" noise="${imu_noise}" />
-    <xacro:gps_sensor parent="rear_axis_center" gps_name="gps" gps_topic="gps/fix" mass="${gps_mass}" sizex="0.03" sizey="0.03" sizez="0.005" ox="0.62" oy="0.25" oz="1.00" update_rate="${gps_update_rate}" initial_latitude="${gps_latitude}" initial_longitude="${gps_longitude}" noise="${gps_noise}" />
+    <xacro:imu_sensor parent="rear_axis_center" imu_name="imu" imu_topic="imu/data_raw" mass="${imu_mass}" sizex="0.03" sizey="0.03" sizez="0.005" ox="0.62" oy="0.25" oz="1.00" update_rate="${imu_update_rate}" noise="${imu_noise}" />
+    <xacro:gps_sensor parent="rear_axis_center" gps_name="gps" gps_topic="gps/fix" mass="${gps_mass}" sizex="0.03" sizey="0.03" sizez="0.005" ox="0.0" oy="0.0" oz="1.365" update_rate="${gps_update_rate}" initial_latitude="${gps_latitude}" initial_longitude="${gps_longitude}" noise="${gps_noise}" />
     <xacro:lidar_sensor parent="rear_axis_center" lidar_name="right_lidar" length="${lidar_length}" radius="${lidar_radius}" mass="${lidar_mass}" ox="1.05" oy="-0.33" oz="0.3" update_rate="${lidar_update_rate}" min_angle="${lidar_min_angle}" max_angle="${lidar_max_angle}" min_range="${lidar_min_range}" max_range="${lidar_max_range}" range_resolution="${lidar_range_resolution}" stdv="${lidar_stdv}" />
     <xacro:lidar_sensor parent="rear_axis_center" lidar_name="left_lidar" length="${lidar_length}" radius="${lidar_radius}" mass="${lidar_mass}" ox="1.05" oy="0.33" oz="0.3" update_rate="${lidar_update_rate}" min_angle="${lidar_min_angle}" max_angle="${lidar_max_angle}" min_range="${lidar_min_range}" max_range="${lidar_max_range}" range_resolution="${lidar_range_resolution}" stdv="${lidar_stdv}" />

File: src/hakuroukun_description/urdf/properties.xacro (robot description, xacro)
@@ -33,10 +33,10 @@
   <xacro:property name="imu_update_rate" value="40.0" />
   <xacro:property name="imu_mass" value="0.05" />
-  <xacro:property name="imu_noise" value="0.001" />
+  <xacro:property name="imu_noise" value="0.0001" />
   <xacro:property name="gps_update_rate" value="10.0" />
   <xacro:property name="gps_mass" value="0.05" />
-  <xacro:property name="gps_noise" value="0.001" />
-  <xacro:property name="gps_latitude" value="34.835190564394" />
-  <xacro:property name="gps_longitude" value="137.45711512765206" />
+  <xacro:property name="gps_noise" value="0.0001" />
+  <xacro:property name="gps_latitude" value="34.70242845166667" />
+  <xacro:property name="gps_longitude" value="137.408935105" />
   <xacro:property name="lidar_update_rate" value="10.0" />			<!-- update rate in ms or in Hz??? -->
   <xacro:property name="lidar_mass" value="0.3" />

Commit message: :+1: update ground truth

File: src/hakuroukun_description/urdf/hakuroukun.urdf.xacro (robot description, xacro)
@@ -100,4 +100,5 @@
     <xacro:lidar_sensor parent="rear_axis_center" lidar_name="right_lidar" length="${lidar_length}" radius="${lidar_radius}" mass="${lidar_mass}" ox="1.05" oy="-0.33" oz="0.3" update_rate="${lidar_update_rate}" min_angle="${lidar_min_angle}" max_angle="${lidar_max_angle}" min_range="${lidar_min_range}" max_range="${lidar_max_range}" range_resolution="${lidar_range_resolution}" stdv="${lidar_stdv}" />
     <xacro:lidar_sensor parent="rear_axis_center" lidar_name="left_lidar" length="${lidar_length}" radius="${lidar_radius}" mass="${lidar_mass}" ox="1.05" oy="0.33" oz="0.3" update_rate="${lidar_update_rate}" min_angle="${lidar_min_angle}" max_angle="${lidar_max_angle}" min_range="${lidar_min_range}" max_range="${lidar_max_range}" range_resolution="${lidar_range_resolution}" stdv="${lidar_stdv}" />
+    <xacro:ground_truth parent="base_link" sizex="0.01" sizey="0.01" sizez="0.01" ox="0.0" oy="0.0" oz="0.01" mass="1"/>
 <!-- ////////////////////////////// GAZEBO ROS PLUGIN //////////////////////////////////// -->
     <gazebo>

File: src/hakuroukun_description/urdf/sensors.xacro (robot description, xacro)
@@ -122,3 +122,27 @@
     </gazebo>
   </xacro:macro>
+  <xacro:macro name="ground_truth" params="parent sizex sizey sizez ox oy oz mass">
+    <link name="ground_truth">
+      <visual>
+        <geometry>
+          <box size="${sizex} ${sizey} ${sizez}"/>
+      </geometry>
+      <material name="White"/>
+      </visual>
+      <xacro:inertial_box mass="${mass}" x="${sizex}" y="${sizey}" z="${sizez}" />
+    </link>
+    <joint name="ground_truth_to_${parent}" type="fixed">
+      <parent link="${parent}"/>
+      <child link="ground_truth"/>
+      <origin xyz="${ox} ${oy} ${oz}"/>
+    </joint>
+    <gazebo>
+      <plugin name="ground_truth" filename="libgazebo_ros_p3d.so">
+        <bodyName>ground_truth</bodyName>
+        <frameName>map</frameName>
+        <updateRate>100.0</updateRate>
+        <topicName>ground_truth/odometry</topicName>
+      </plugin>
+    </gazebo>
+  </xacro:macro>
 </robot>

Commit message: :+1: update launch files

File: src/hakuroukun_description/urdf/hakuroukun.urdf.xacro (robot description, xacro)
@@ -98,6 +98,6 @@
     <xacro:imu_sensor parent="rear_axis_center" imu_name="imu" imu_topic="imu/data_raw" mass="${imu_mass}" sizex="0.03" sizey="0.03" sizez="0.005" ox="0.62" oy="-0.25" oz="1.00" update_rate="${imu_update_rate}" noise="${imu_noise}" />
     <xacro:gps_sensor parent="rear_axis_center" gps_name="gps" gps_topic="fix" mass="${gps_mass}" sizex="0.03" sizey="0.03" sizez="0.005" ox="0.6" oy="0.0" oz="1.365" update_rate="${gps_update_rate}" initial_latitude="${gps_latitude}" initial_longitude="${gps_longitude}" noise="${gps_noise}" />
-    <xacro:lidar_sensor parent="rear_axis_center" lidar_name="right_lidar" length="${lidar_length}" radius="${lidar_radius}" mass="${lidar_mass}" ox="1.05" oy="-0.33" oz="0.3" update_rate="${lidar_update_rate}" min_angle="${lidar_min_angle}" max_angle="${lidar_max_angle}" min_range="${lidar_min_range}" max_range="${lidar_max_range}" range_resolution="${lidar_range_resolution}" stdv="${lidar_stdv}" />
-    <xacro:lidar_sensor parent="rear_axis_center" lidar_name="left_lidar" length="${lidar_length}" radius="${lidar_radius}" mass="${lidar_mass}" ox="1.05" oy="0.33" oz="0.3" update_rate="${lidar_update_rate}" min_angle="${lidar_min_angle}" max_angle="${lidar_max_angle}" min_range="${lidar_min_range}" max_range="${lidar_max_range}" range_resolution="${lidar_range_resolution}" stdv="${lidar_stdv}" />
+    <xacro:lidar_sensor parent="rear_axis_center" lidar_name="right_lidar" length="${lidar_length}" radius="${lidar_radius}" mass="${lidar_mass}" ox="1.05" oy="-0.33" oz="0.3" roll="0" pitch="0" yaw="${pi}" update_rate="${lidar_update_rate}" min_angle="${lidar_min_angle}" max_angle="${lidar_max_angle}" min_range="${lidar_min_range}" max_range="${lidar_max_range}" range_resolution="${lidar_range_resolution}" stdv="${lidar_stdv}" />
+    <xacro:lidar_sensor parent="rear_axis_center" lidar_name="left_lidar" length="${lidar_length}" radius="${lidar_radius}" mass="${lidar_mass}" ox="1.05" oy="0.33" oz="0.3" roll="0" pitch="0" yaw="${pi}" update_rate="${lidar_update_rate}" min_angle="${lidar_min_angle}" max_angle="${lidar_max_angle}" min_range="${lidar_min_range}" max_range="${lidar_max_range}" range_resolution="${lidar_range_resolution}" stdv="${lidar_stdv}" />
     <xacro:ground_truth parent="base_link" sizex="0.01" sizey="0.01" sizez="0.01" ox="0.0" oy="0.0" oz="0.01" mass="1"/>
 <!-- ////////////////////////////// GAZEBO ROS PLUGIN //////////////////////////////////// -->

File: src/hakuroukun_description/urdf/sensors.xacro (robot description, xacro)
@@ -68,5 +68,5 @@
 	</gazebo>
 	</xacro:macro>
-  <xacro:macro name="lidar_sensor" params="parent lidar_name length radius mass ox oy oz update_rate min_angle max_angle min_range max_range range_resolution stdv" >
+  <xacro:macro name="lidar_sensor" params="parent lidar_name length radius mass ox oy oz roll pitch yaw update_rate min_angle max_angle min_range max_range range_resolution stdv" >
     <link name="${lidar_name}">
       <visual>
@@ -74,5 +74,5 @@
           <cylinder length="${length}" radius="${radius}"/>
         </geometry>
-        <origin rpy="0 0 0" xyz="0 0 0"/>
+        <origin rpy="${roll} ${pitch} ${yaw}" xyz="0 0 0"/>
         <material name="Black"/>
       </visual>
@@ -84,5 +84,5 @@
     <joint name="$[parent}_to_${lidar_name}" type="fixed">
       <parent link="${parent}"/>
-        <child link="${lidar_name}"/>
+      <child link="${lidar_name}"/>
       <origin xyz="${ox} ${oy} ${oz}"/>
     </joint>

Commit message: :+1: update camera sensor

File: src/hakuroukun_description/urdf/hakuroukun.urdf.xacro (robot description, xacro)
@@ -101,4 +101,5 @@
     <xacro:lidar_sensor parent="rear_axis_center" lidar_name="left_lidar" length="${lidar_length}" radius="${lidar_radius}" mass="${lidar_mass}" ox="1.05" oy="0.33" oz="0.3" roll="0" pitch="0" yaw="${pi}" update_rate="${lidar_update_rate}" min_angle="${lidar_min_angle}" max_angle="${lidar_max_angle}" min_range="${lidar_min_range}" max_range="${lidar_max_range}" range_resolution="${lidar_range_resolution}" stdv="${lidar_stdv}" />
     <xacro:ground_truth parent="base_link" sizex="0.01" sizey="0.01" sizez="0.01" ox="0.0" oy="0.0" oz="0.01" mass="1"/>
+    <xacro:camera_sensor parent="rear_axis_center" camera_name="camera" mass="0.1" sizex="0.03" sizey="0.1" sizez="0.03" ox="1.2" oy="0.0" oz="0.8"/>
 <!-- ////////////////////////////// GAZEBO ROS PLUGIN //////////////////////////////////// -->
     <gazebo>

File: src/hakuroukun_description/urdf/sensors.xacro (robot description, xacro)
@@ -147,3 +147,45 @@
     </gazebo>
   </xacro:macro>
+  <xacro:macro name="camera_sensor" params="parent camera_name mass ox oy oz sizex sizey sizez">
+    <link name="${camera_name}">
+      <visual>
+        <geometry>
+          <box size="${sizex} ${sizey} ${sizez}"/>
+        </geometry>
+        <material name="White"/>
+      </visual>
+      <xacro:inertial_box mass="${mass}" x="${sizex}" y="${sizey}" z="${sizez}" />
+    </link>
+    <joint name="${parent}_to_${camera_name}" type="fixed">
+      <parent link="${parent}"/>
+      <child link="${camera_name}"/>
+      <origin xyz="${ox} ${oy} ${oz}"/>
+    </joint>
+    <gazebo reference="${camera_name}">
+       <sensor type="camera" name="${camera_name}_camera">
+        <always_on>true</always_on>
+        <update_rate>30.0</update_rate>
+        <visualize>true</visualize>
+        <camera name="${camera_name}_camera">
+          <horizontal_fov>1.3962634</horizontal_fov>
+          <image>
+            <width>640</width>
+            <height>480</height>
+            <format>R8G8B8</format>
+          </image>
+          <clip>
+            <near>0.1</near>
+            <far>100</far>
+          </clip>
+        </camera>
+        <plugin name="camera_controller" filename="libgazebo_ros_camera.so">
+          <updateRate>30.0</updateRate>
+          <cameraName>${camera_name}_camera</cameraName>
+          <imageTopicName>${camera_name}/image_raw</imageTopicName>
+          <cameraInfoTopicName>${camera_name}/camera_info</cameraInfoTopicName>
+          <frameName>${camera_name}</frameName>
+        </plugin>
+      </sensor>
+    </gazebo>
+  </xacro:macro>
 </robot>

Commit message: add code for tasp with cone

File: src/hakuroukun_description/urdf/hakuroukun.urdf.xacro (robot description, xacro)
@@ -115,6 +115,6 @@
     <xacro:imu_sensor parent="rear_axis_center" imu_name="imu" imu_topic="imu/data_raw" mass="${imu_mass}" sizex="0.03" sizey="0.03" sizez="0.005" ox="0.62" oy="-0.25" oz="${1.00-rear_radius}" update_rate="${imu_update_rate}" noise="${imu_noise}" />
     <xacro:gps_sensor parent="rear_axis_center" gps_name="gps" gps_topic="fix" mass="${gps_mass}" sizex="0.03" sizey="0.03" sizez="0.005" ox="0.6" oy="0.0" oz="${1.365-rear_radius}" update_rate="${gps_update_rate}" initial_latitude="${gps_latitude}" initial_longitude="${gps_longitude}" noise="${gps_noise}" />
-    <xacro:lidar_sensor parent="rear_axis_center" lidar_name="right_lidar" length="${lidar_length}" radius="${lidar_radius}" mass="${lidar_mass}" ox="1.03" oy="-0.31" oz="${0.365-rear_radius}" roll="0" pitch="0" yaw="${pi}" update_rate="${lidar_update_rate}" min_angle="${lidar_min_angle}" max_angle="${lidar_max_angle}" min_range="${lidar_min_range}" max_range="${lidar_max_range}" range_resolution="${lidar_range_resolution}" stdv="${lidar_stdv}" />
-    <xacro:lidar_sensor parent="rear_axis_center" lidar_name="left_lidar" length="${lidar_length}" radius="${lidar_radius}" mass="${lidar_mass}" ox="1.03" oy="0.31" oz="${0.365-rear_radius}" roll="0" pitch="0" yaw="${pi}" update_rate="${lidar_update_rate}" min_angle="${lidar_min_angle}" max_angle="${lidar_max_angle}" min_range="${lidar_min_range}" max_range="${lidar_max_range}" range_resolution="${lidar_range_resolution}" stdv="${lidar_stdv}" />
+    <xacro:lidar_sensor parent="rear_axis_center" lidar_name="right_lidar" length="${lidar_length}" radius="${lidar_radius}" mass="${lidar_mass}" ox="1.03" oy="-0.31" oz="${0.365-rear_radius+0.05}" roll="0" pitch="0" yaw="${pi}" update_rate="${lidar_update_rate}" min_angle="${lidar_min_angle}" max_angle="${lidar_max_angle}" min_range="${lidar_min_range}" max_range="${lidar_max_range}" range_resolution="${lidar_range_resolution}" stdv="${lidar_stdv}" />
+    <xacro:lidar_sensor parent="rear_axis_center" lidar_name="left_lidar" length="${lidar_length}" radius="${lidar_radius}" mass="${lidar_mass}" ox="1.03" oy="0.31" oz="${0.365-rear_radius+0.05}" roll="0" pitch="0" yaw="${pi}" update_rate="${lidar_update_rate}" min_angle="${lidar_min_angle}" max_angle="${lidar_max_angle}" min_range="${lidar_min_range}" max_range="${lidar_max_range}" range_resolution="${lidar_range_resolution}" stdv="${lidar_stdv}" />
     <xacro:ground_truth parent="base_link" sizex="0.01" sizey="0.01" sizez="0.01" ox="0.0" oy="0.0" oz="0.01" mass="1"/>
     <xacro:zed2_camera camera_name="camera_link" parent="rear_axis_center" mass="0.06" ox="1.01" oy="0.0" oz="${1.195-rear_radius}" roll="0" pitch="0" yaw="0" />

File: src/hakuroukun_description/urdf/properties.xacro (robot description, xacro)
@@ -6,5 +6,5 @@
   <xacro:property name="robot_width" value="0.810" />
   <xacro:property name="robot_height" value="1.070" />
-  <xacro:property name="robot_mass" value="270" />
+  <xacro:property name="robot_mass" value="304" />
   <!-- ///////////////////////////////////////////////////////////// -->
   <!-- /////////////////// Base link to Robot frame /////////////////// -->
@@ -33,8 +33,8 @@
   <xacro:property name="imu_update_rate" value="40.0" />
   <xacro:property name="imu_mass" value="0.05" />
-  <xacro:property name="imu_noise" value="0.0" />
+  <xacro:property name="imu_noise" value="0.01" />
   <xacro:property name="gps_update_rate" value="40.0" />
   <xacro:property name="gps_mass" value="0.05" />
-  <xacro:property name="gps_noise" value="0.0" />
+  <xacro:property name="gps_noise" value="0.01" />
   <xacro:property name="gps_latitude" value="34.70242845166667" />
   <xacro:property name="gps_longitude" value="137.408935105" />

File: src/hakuroukun_description/urdf/sensors.xacro (robot description, xacro)
@@ -77,5 +77,5 @@
           <cylinder length="${length}" radius="${radius}"/>
         </geometry>
-        <origin xyz="0 0 0.05"/>
+        <origin xyz="0 0 0"/>
         <material name="DarkGrey"/>
       </visual>
