Commit message: modify code to use with gmapping

File: src/hakuroukun_description/urdf/hakuroukun.urdf.xacro (robot description, xacro)
@@ -71,5 +71,5 @@
     </joint>
     <!-- lidar center-->
-    <link name="lidar_center">
+    <link name="laser_link">
         <visual>
         <geometry>
@@ -79,10 +79,10 @@
         </visual>
     </link>
-    <gazebo reference="lidar_center">
+    <gazebo reference="laser_link">
         <material>Gazebo/Red</material>
     </gazebo>
-    <joint name="rear_axis_center_to_lidar_center" type="fixed">
+    <joint name="laser_link" type="fixed">
         <parent link="rear_axis_center" />
-        <child link="lidar_center" />
+        <child link="laser_link" />
         <origin xyz="1.03 0.0 ${0.365-rear_radius}" />
     </joint>

File: src/hakuroukun_description/urdf/properties.xacro (robot description, xacro)
@@ -44,5 +44,5 @@
   <xacro:property name="lidar_radius" value="0.038" />
   <xacro:property name="lidar_min_range" value="0.2" />
-  <xacro:property name="lidar_max_range" value="8.0" />
+  <xacro:property name="lidar_max_range" value="25.0" />
   <xacro:property name="lidar_stdv" value="0.01" />
   <xacro:property name="lidar_range_resolution" value="0.01" />
