Commit message: :+1: update sensor rotation and pose

File: src/hakuroukun_description/urdf/properties.xacro (robot description, xacro)
@@ -36,5 +36,5 @@
   <xacro:property name="gps_update_rate" value="10.0" />
   <xacro:property name="gps_mass" value="0.05" />
-  <xacro:property name="gps_noise" value="0.05" />
+  <xacro:property name="gps_noise" value="0.01" />
   <xacro:property name="gps_latitude" value="34.70242845166667" />
   <xacro:property name="gps_longitude" value="137.408935105" />

Commit message: update code

File: src/hakuroukun_description/urdf/properties.xacro (robot description, xacro)
@@ -13,5 +13,5 @@
   <xacro:property name="base_link_to_robot_frame_Z" value="0.440" />
   <!-- /////////////////// Steering Unit /////////////////// -->
-  <xacro:property name="rear_axis_center_to_steering_center" value="1.1" /> <!-- approx. value -->
+  <xacro:property name="rear_axis_center_to_steering_center" value="1.0" /> <!-- approx. value -->
   <xacro:property name="steering_X" value="0.3" />
   <xacro:property name="steering_Y" value="0.2" />
